File: electrical/TwoMonth_ProjectFlyingPenguin.sch (KiCad schematic (older format))
At the start: 11 parts, among them J1 USB_B_Micro, J2 Conn_ARM_JTAG_SWD_10, J3 Micro_SD_Card_Det, M1 Elevator_Servo, M2 Fin_Servo, U1 ATSAMD21G18A-AUT, U2 AT25SF081-XMHD-X, U3 BNO055, U4 MS561101BA03-50, Y1 Crystal

Commit message: Added power part of schematic. doing mcu now
Parts:
- removed J?: VBatt, symbol Connector:Barrel_Jack_Switch
- removed Y1: Crystal, Crystal:Crystal_AT310_D3.0mm_L10.0mm_Horizontal_1EP_style2, symbol Device:Crystal
- added C?: 0.47uF, symbol Device:C_Small
- added C?: 22uF, symbol Device:C_Small
- added C? (x2): 1nF, symbol Device:C_Small
- added C? (x2): 10uF, symbol Device:C_Small
- added C? (x2): 6.8pF, symbol Device:C_Small
- added D?: PRTR5V0U2X_215, digikey-footprints:TO-253-4, symbol dk_TVS-Diodes:PRTR5V0U2X_215
- added FB?: 470 @ 100Mhz, symbol Device:Ferrite_Bead_Small
- added J?: Barrel_Jack_Switch, symbol Connector:Barrel_Jack_Switch
- added Q?: PFETDefaultA, digikey-footprints:TO-220-3, symbol dk_Transistors-FETs-MOSFETs-Single:FQP27P06
- added Q?: PFETDefaultB, digikey-footprints:TO-220-3, symbol dk_Transistors-FETs-MOSFETs-Single:FQP27P06
- added Q?: PFETAltB, digikey-footprints:TO-220-3, symbol dk_Transistors-FETs-MOSFETs-Single:FQP27P06
- added Q?: PFETAltA, digikey-footprints:TO-220-3, symbol dk_Transistors-FETs-MOSFETs-Single:FQP27P06
- added R? (x2): 200K, symbol Device:R_Small
- added R?: 100K, symbol Device:R_Small
- added U?: LM2940_TO220, Package_TO_SOT_THT:TO-220-3_Vertical, symbol Regulator_Linear:LM7805_TO220
- added U?: MIC29310, Package_TO_SOT_THT:TO-220-3_Vertical, symbol Regulator_Linear:LM7805_TO220
- added Y?: 32.768kHz, symbol Device:Crystal_GND2_Small
- J2: symbol Connector:Conn_ARM_JTAG_SWD_10 -> TwoMonth_ProjectFlyingPenguin-rescue:Conn_ARM_JTAG_SWD_10-Connector
- J3: symbol Connector:Micro_SD_Card_Det -> TwoMonth_ProjectFlyingPenguin-rescue:Micro_SD_Card_Det-Connector
Connections:
- net labels added: +3V3, +5V, GND, USB_5V+, USB_D+, USB_D-, XIN32, XOUT32
- wire segments 0 -> 91
- no-connect marks 0 -> 1
Other:
- moved on the sheet: U1, U2

Commit message: Finished placing parts. need to route tracks
Parts:
- removed Y?: 32.768kHz, symbol Device:Crystal_GND2_Small
- added C10, C12, C13, C15: 100nF, Capacitor_SMD:C_0603_1608Metric_Pad1.05x0.95mm_HandSolder, symbol Device:C_Small
- added C11: 1uF, Capacitor_SMD:C_0603_1608Metric_Pad1.05x0.95mm_HandSolder, symbol Device:C_Small
- added C14: 10uF, Capacitor_SMD:C_0603_1608Metric_Pad1.05x0.95mm_HandSolder, symbol Device:C_Small
- added C16, C17: 0.1uF, Capacitor_SMD:C_0603_1608Metric_Pad1.05x0.95mm_HandSolder, symbol Device:C_Small
- added C18, C19: 22pF, Capacitor_SMD:C_0603_1608Metric_Pad1.05x0.95mm_HandSolder, symbol Device:C_Small
- added C9: 4F, Battery:SuperCap, symbol Device:CP
- added D2: POWER_LED, symbol Device:LED
- added FB2: 470 @ 100Mhz (BLM18PG471SN1), Capacitor_SMD:C_0603_1608Metric_Pad1.05x0.95mm_HandSolder, symbol Device:Ferrite_Bead_Small
- added J5: Hotwire, Connector_PinHeader_2.54mm:PinHeader_1x02_P2.54mm_Vertical, symbol Connector:Conn_01x02_Female
- added Q5: FQP27P06, digikey-footprints:TO-220-3, symbol dk_Transistors-FETs-MOSFETs-Single:FQP27P06
- added Q6: FQP30N06L, digikey-footprints:TO-220-3, symbol dk_Transistors-FETs-MOSFETs-Single:FQP30N06L
- added R10, R11, R12, R13, R4, R5, R6, R7, R8: 10k, Resistor_SMD:R_0603_1608Metric_Pad1.05x0.95mm_HandSolder, symbol Device:R_Small
- added R14: 330, symbol Device:R_Small
- added R9: 1k, Resistor_SMD:R_0603_1608Metric_Pad1.05x0.95mm_HandSolder, symbol Device:R_Small
- added Y1, Y2: 32.768Khz, Crystal:Crystal_SMD_MicroCrystal_MS1V-T1K, symbol Device:Crystal_GND3_Small
- C1, C2, C3, C4, C5, C6, C7, C8: renamed from C?; footprint (none) -> Capacitor_SMD:C_0603_1608Metric_Pad1.05x0.95mm_HandSolder
- FB1: renamed from FB?; value 470 @ 100Mhz -> 470 @ 100Mhz (BLM18PG471SN1); footprint (none) -> Capacitor_SMD:C_0603_1608Metric_Pad1.05x0.95mm_HandSolder
- J4: renamed from J?; value Barrel_Jack_Switch -> Battery_Barrel_Jack; footprint (none) -> Connector_BarrelJack:BarrelJack_Horizontal
- R1, R2, R3: renamed from R?; footprint (none) -> Resistor_SMD:R_0603_1608Metric_Pad1.05x0.95mm_HandSolder
- gave numbers to parts that had none: 7
Connections:
- net +3V3: now also J2.1 (VCC), J3.4 (VDD), U1.17 (VDD/IO), U1.36 (VDD/IO), U1.43 (VDDCORE), U1.44 (VDDIN), U2.8 (VCC), U3.28 (VDDIO), U3.3 (VDD), U3.4 (~nBOOT_LOAD_PIN), U4.1 (VDD), C10.1, C11.1, C12.1, C13.1, C16.1, D2.2 (A), FB2.1, R10.2, R4.2, R5.2, R7.1, R8.1, R9.1
- net +5V: now also M1.2 (+), M2.2 (+), Q5.3 (S)
- net GND: now also J2.3 (GND), J2.5 (GND), J2.9 (GNDDetect), J3.11 (SHIELD), J3.6 (VSS), M1.3 (-), M2.3 (-), U2.4 (GND), U3.10 (BL_IND), U3.15 (GNDIO), U3.16 (GNDIO), U3.18 (COM2), U3.2 (GND), U3.25 (GNDIO), U4.3 (GND), C10.2, C11.2, C12.2, C13.2, C14.2, C15.2, C16.2, C17.2, C18.2, C19.1, C9.2, Q6.3 (S), R11.2, R12.2, R13.2, R14.2, R6.2, Y1.3
- net XIN32: now also Y1.1
- net XOUT32: now also Y1.2
- net SPI0_SS_0: now reaches U1.10 (PA05)
- net SPI0_SS_0: now also U2.1 (~CS)
- net SPI0_MOSI: now reaches U1.11 (PA06)
- net SPI0_MOSI: now also J3.3 (CMD), J3.7 (DAT0), U2.2 (SO/IO1), U2.5 (SI/IO0)
- net SPI0_SCK: now reaches U1.12 (PA07)
- net SPI0_SCK: now also J3.5 (CLK), U2.6 (SCK)
- net SDA: now reaches U1.13 (PA08)
- net SDA: now also U3.20 (COM0), U4.7 (SDI/SDA), R7.2
- net SCL: now reaches U1.14 (PA09)
- net SCL: now also U3.19 (COM1), U4.8 (SCLK), R8.2
- net PWM1_ELEV: now reaches U1.15 (PA10)
- net PWM1_ELEV: now also M1.1 (PWM)
- net Hotwire_GPO: now reaches U1.16 (PA11)
- net Hotwire_GPO: now also Q5.1 (G), Q6.1 (G), R6.1
- net PWM0_FIN: now reaches U1.19 (PB10)
- net PWM0_FIN: now also M2.1 (PWM)
- net SPI0_SS_1: now reaches U1.21 (PA12)
- net SPI0_SS_1: now also J3.2 (DAT3/CD)
- net uSD_CARD_DET: now reaches U1.22 (PA13)
- net uSD_CARD_DET: now also J3.10 (DET_A)
- net BATTV_ADC0: now reaches U1.3 (PA02)
- net FLIGHT_LED_2: now reaches U1.37 (PB22)
- net THERM1_ADC1: now reaches U1.4 (PA03)
- net ~MCU_RESET: now reaches U1.40 (~RESET)
- net ~MCU_RESET: now also U3.11 (~nRESET)
- net SWCLK: now reaches U1.45 (PA30)
- net SWCLK: now also J2.4 (SWDCLK/TCK), R9.2
- net SWDIO: now reaches U1.46 (PA31)
- net SWDIO: now also J2.2 (SWDIO/TMS)
- net VDD_ANA: now reaches U1.6 (VDD/ANA)
- net VDD_ANA: now also C14.1, C15.1, FB2.2
- net FLIGHT_LED_0: now reaches U1.7 (PB08)
- net FLIGHT_LED_1: now reaches U1.8 (PB09)
- net SPI0_MISO: now reaches U1.9 (PA04)
- net at U2.3 (~WP~/IO2): now also R4.1
- net at U2.7 (~HOLD~/IO3): now also R5.1
- net at U3.17 (COM3): now also R11.1
- net BNO_XOUT32: now reaches U3.26 (XOUT32)
- net BNO_XOUT32: now also C18.1, Y2.2
- net BNO_XIN32: now reaches U3.27 (XIN32)
- net BNO_XIN32: now also C19.2, Y2.1
- net at U3.5 (PS1): now also R12.1
- net at U3.6 (PS0): now also R13.1
- net at U3.9 (CAP): now also C17.1
- net at U4.2 (PS): now also U4.4 (~CSB~), U4.5 (~CSB~), R10.1
- net VBUS: now reaches C2.1, D1.4 (VCC), FB1.2, J1.1 (VBUS)
- net ~SYS_RESET: now reaches J2.10 (~RESET~)
- new net: J5.2 (Pin_2), Q6.2 (D)
- new net: C9.1, J5.1 (Pin_1), Q5.2 (D)
- new net: D2.1 (K), R14.1
- no-connect marks 1 -> 8
Other:
- note added: "32.768 Crystal Oscillator\n"
- note added: "BRAIN"
- note added: "Flash Memory"
- note added: "HOTWIRE"
- note added: "MCU"
- note added: "POWER"
- note added: "Pullup Resistors for I2C"
- note added: "SENSORS"
- note added: "SERVOS"
- note added: "SWD (Debugger)"
- moved on the sheet: C1, C3, C5, C6, C7, C8, J2, J3, J4, M1, M2, Q1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

Commit message: Finished schematic I think. Cant find part for rbf switch
Parts:
- added J10: NTCLE100E3103JB0 (Therm 1), Connector_PinHeader_2.54mm:PinHeader_1x02_P2.54mm_Vertical, symbol Connector:Conn_01x02_Male
- added J11: NTCLE100E3103JB0 (Therm 2), Connector_PinHeader_2.54mm:PinHeader_1x02_P2.54mm_Vertical, symbol Connector:Conn_01x02_Male
- added J6: FLIGHT_LED_0, Connector_PinHeader_2.54mm:PinHeader_1x02_P2.54mm_Vertical, symbol Connector:Conn_01x02_Female
- added J7: SS0750301F020P1A, Button_Switch_THT:Push_E-Switch_KS01Q01, symbol FlyingPenguin:SS0750301F020P1A
- added J8: FLIGHT_LED_1, Connector_PinHeader_2.54mm:PinHeader_1x02_P2.54mm_Vertical, symbol Connector:Conn_01x02_Female
- added J9: FLIGHT_LED_2, Connector_PinHeader_2.54mm:PinHeader_1x02_P2.54mm_Vertical, symbol Connector:Conn_01x02_Female
- added Q7: FQP30N06L, digikey-footprints:TO-220-3, symbol dk_Transistors-FETs-MOSFETs-Single:FQP30N06L
- added R15, R17, R18: 25, Resistor_SMD:R_0603_1608Metric_Pad1.05x0.95mm_HandSolder, symbol Device:R_Small
- added R16: 4.7k, Resistor_SMD:R_0603_1608Metric_Pad1.05x0.95mm_HandSolder, symbol Device:R_Small
- added R19: 100k, Resistor_SMD:R_0603_1608Metric_Pad1.05x0.95mm_HandSolder, symbol Device:R_Small
- added R20: 39, Resistor_SMD:R_0603_1608Metric_Pad1.05x0.95mm_HandSolder, symbol Device:R_Small
- added R21: 10k, Resistor_SMD:R_0603_1608Metric_Pad1.05x0.95mm_HandSolder, symbol Device:R_Small
- added R22: 3.2k, Resistor_SMD:R_0603_1608Metric_Pad1.05x0.95mm_HandSolder, symbol Device:R_Small
- added R23, R24: 20k, Resistor_SMD:R_0603_1608Metric_Pad1.05x0.95mm_HandSolder, symbol Device:R_Small
- added S1: ~RESET_BUTTON, digikey-footprints:PushButton_12x12mm_THT_GPTS203211B, symbol dk_Pushbutton-Switches:GPTS203211B
- D2: footprint (none) -> LED_SMD:LED_0603_1608Metric_Pad1.05x0.95mm_HandSolder
- R14: footprint (none) -> Resistor_SMD:R_0603_1608Metric_Pad1.05x0.95mm_HandSolder
- Y1, Y2: symbol Device:Crystal_GND3_Small -> TwoMonth_ProjectFlyingPenguin-rescue:Crystal_GND3_Small-Device
Connections:
- net ~MCU_RESET is gone; now on net ~SYS_RESET: U1.40 (~RESET), U3.11 (~nRESET)
- net +3V3: now also R15.2, R17.2, R18.2, R19.1, R23.1, R24.1
- net BATTV_ADC0: now also R21.2, R22.1
- net GND: now also Y2.3, J10.1 (Pin_1), J11.1 (Pin_1), Q7.3 (S), R16.1, R22.2, S1.2
- net THERM1_ADC1: now also J10.2 (Pin_2), R23.2
- net ~SYS_RESET: now also R19.2, R20.1
- net RAW_BATTERY_V+: now reaches C1.1, U5.1 (VI)
- net RAW_BATTERY_V+: now also J7.1 (COM), R21.1; no longer J4.1
- net FLIGHT_LED_0 renamed THERM2_ADC2
- net THERM2_ADC2: now also J11.2 (Pin_2), R24.2
- net FLIGHT_LED_1: no longer names the net of U1.8 (PB09)
- net FLIGHT_LED_2 renamed FLIGHT_LED_CTRL
- net FLIGHT_LED_CTRL: now also Q7.1 (G), R16.2
- new net: J4.1, J7.3 (NC)
- new net: R20.2, S1.1
- new net: J6.1 (Pin_1), R15.1
- new net: J8.1 (Pin_1), R17.1
- new net: J9.1 (Pin_1), R18.1
- new net FLIGHT_LED_DRAIN: J6.2 (Pin_2), J8.2 (Pin_2), J9.2 (Pin_2), Q7.2 (D)
- no-connect marks 8 -> 9
Other:
- note added: "ADC INPUTS"
- note added: "FLIGHT LEDs"
- note added: "nRESET Circuit"
- moved on the sheet: C1, D2, J4, R14
